Commit message: Xacro tag formatting which caused roslaunch `collision_avoidance_pick_and_place ur5_setup.launch` to fail

File: exercises/Perception-Driven_Manipulation/solution_ws/src/robot_config/urdf/ur5.urdf.xacro (robot description, xacro)
@@ -4,17 +4,17 @@
   <xacro:include filename="$(find ur_description)/urdf/ur.gazebo.xacro" />
   <!-- Inertia parameters -->
-  <property name="base_mass" value="4.0" />  <!-- This mass might be incorrect -->
-  <property name="shoulder_mass" value="3.7000" />
-  <property name="upper_arm_mass" value="8.3930" />
-  <property name="forearm_mass" value="2.2750" />
-  <property name="wrist_1_mass" value="1.2190" />
-  <property name="wrist_2_mass" value="1.2190" />
-  <property name="wrist_3_mass" value="0.1879" />
-  <property name="shoulder_cog" value="0.0 0.00193 -0.02561" />
-  <property name="upper_arm_cog" value="0.0 -0.024201 0.2125" />
-  <property name="forearm_cog" value="0.0 0.0265 0.11993" />
-  <property name="wrist_1_cog" value="0.0 0.110949 0.01634" />
-  <property name="wrist_2_cog" value="0.0 0.0018 0.11099" />
-  <property name="wrist_3_cog" value="0.0 0.001159 0.0" />
+  <xacro:property name="base_mass" value="4.0" />  <!-- This mass might be incorrect -->
+  <xacro:property name="shoulder_mass" value="3.7000" />
+  <xacro:property name="upper_arm_mass" value="8.3930" />
+  <xacro:property name="forearm_mass" value="2.2750" />
+  <xacro:property name="wrist_1_mass" value="1.2190" />
+  <xacro:property name="wrist_2_mass" value="1.2190" />
+  <xacro:property name="wrist_3_mass" value="0.1879" />
+  <xacro:property name="shoulder_cog" value="0.0 0.00193 -0.02561" />
+  <xacro:property name="upper_arm_cog" value="0.0 -0.024201 0.2125" />
+  <xacro:property name="forearm_cog" value="0.0 0.0265 0.11993" />
+  <xacro:property name="wrist_1_cog" value="0.0 0.110949 0.01634" />
+  <xacro:property name="wrist_2_cog" value="0.0 0.0018 0.11099" />
+  <xacro:property name="wrist_3_cog" value="0.0 0.001159 0.0" />
   <!-- Kinematic model -->
   <!-- Properties from urcontrol.conf -->
@@ -29,20 +29,20 @@
     center_of_mass = [ [0, -0.02561, 0.00193], [0.2125, 0, 0.11336], [0.11993, 0.0, 0.0265], [0, -0.0018, 0.01634], [0, 0.0018,0.01634], [0, 0, -0.001159] ]
   -->
-  <property name="ur5_d1" value="0.089159" />
-  <property name="ur5_a2" value="-0.42500" />
-  <property name="ur5_a3" value="-0.39225" />
-  <property name="ur5_d4" value="0.10915" />
-  <property name="ur5_d5" value="0.09465" />
-  <property name="ur5_d6" value="0.0823" />
+  <xacro:property name="ur5_d1" value="0.089159" />
+  <xacro:property name="ur5_a2" value="-0.42500" />
+  <xacro:property name="ur5_a3" value="-0.39225" />
+  <xacro:property name="ur5_d4" value="0.10915" />
+  <xacro:property name="ur5_d5" value="0.09465" />
+  <xacro:property name="ur5_d6" value="0.0823" />
   <!-- Arbitrary offsets for shoulder/elbow joints -->
-  <property name="shoulder_offset" value="0.13585" />  <!-- measured from model -->
-  <property name="elbow_offset" value="-0.1197" /> <!-- measured from model -->
+  <xacro:property name="shoulder_offset" value="0.13585" />  <!-- measured from model -->
+  <xacro:property name="elbow_offset" value="-0.1197" /> <!-- measured from model -->
   <!-- link lengths used in model -->
-  <property name="shoulder_height" value="${ur5_d1}" />
-  <property name="upper_arm_length" value="${-ur5_a2}" />
-  <property name="forearm_length" value="${-ur5_a3}" />
-  <property name="wrist_1_length" value="${ur5_d4 - elbow_offset - shoulder_offset}" />
-  <property name="wrist_2_length" value="${ur5_d5}" />
-  <property name="wrist_3_length" value="${ur5_d6}" />
+  <xacro:property name="shoulder_height" value="${ur5_d1}" />
+  <xacro:property name="upper_arm_length" value="${-ur5_a2}" />
+  <xacro:property name="forearm_length" value="${-ur5_a3}" />
+  <xacro:property name="wrist_1_length" value="${ur5_d4 - elbow_offset - shoulder_offset}" />
+  <xacro:property name="wrist_2_length" value="${ur5_d5}" />
+  <xacro:property name="wrist_3_length" value="${ur5_d6}" />
   <!--property name="shoulder_height" value="0.089159" /-->
   <!--property name="shoulder_offset" value="0.13585" /-->  <!-- shoulder_offset - elbow_offset + wrist_1_length = 0.10915 -->
@@ -53,13 +53,13 @@
   <!--property name="wrist_2_length" value="0.09465" /-->   <!-- In CAD this distance is 0.930, but in the spec it is 0.09465 -->
   <!--property name="wrist_3_length" value="0.0823" /-->
-  <property name="shoulder_radius" value="0.060" />   <!-- manually measured -->
-  <property name="upper_arm_radius" value="0.054" />  <!-- manually measured -->
-  <property name="elbow_radius" value="0.060" />      <!-- manually measured -->
-  <property name="forearm_radius" value="0.040" />    <!-- manually measured -->
-  <property name="wrist_radius" value="0.045" />      <!-- manually measured -->
+  <xacro:property name="shoulder_radius" value="0.060" />   <!-- manually measured -->
+  <xacro:property name="upper_arm_radius" value="0.054" />  <!-- manually measured -->
+  <xacro:property name="elbow_radius" value="0.060" />      <!-- manually measured -->
+  <xacro:property name="forearm_radius" value="0.040" />    <!-- manually measured -->
+  <xacro:property name="wrist_radius" value="0.045" />      <!-- manually measured -->
   <xacro:macro name="cylinder_inertial" params="radius length mass *origin">
     <inertial>
       <mass value="${mass}" />
-      <insert_block name="origin" />
+      <xacro:insert_block name="origin" />
       <inertia ixx="${0.0833333 * mass * (3 * radius * radius + length * length)}" ixy="0.0" ixz="0.0"
         iyy="${0.0833333 * mass * (3 * radius * radius + length * length)}" iyz="0.0"
